File: electronics/u-nit/u-nit.kicad_sch (KiCad schematic)
At the start: 53 parts, among them J1 TBP02R2-381-02BE, J10 TBP02R2-381-04BE, J11 TBP02R2-381-04BE, J12 TBP02R2-381-03BE, J2 PJ-002A, J3 Conn_ARM_JTAG_SWD_10, J4 Conn_01x05_Socket, J5 TBP02R2-381-04BE, J6 TBP02R2-381-03BE, J7 TBP02R2-381-04BE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

Commit message: added digikey BOM, schematic (pdf) and gerber files
Other:
- company: (none) -> Harvey Bates
- title: (none) -> U-NIT
Changed lines of the file:
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@@
 (kicad_sch (version 20230121) (generator eeschema)
   (paper "A4")
+  (title_block
+    (title "U-NIT")
+    (date "2023-08-27")
+    (rev "1.0")
+    (company "Harvey Bates")
+  )
   (junction (at 189.865 132.08) (diameter 0) (color 0 0 0 0)
   )
